Commit message: fixed the frame of force from tool to world

File: install/mujoco_ros2_control_demos/share/mujoco_ros2_control_demos/urdf/fr3_nohand.urdf (robot description, URDF)
Before this commit: robot fr3, 10 links, 9 joints
Links:
- removed link fr3_link8
- added link touch_tip, mass 1e-6; collision sphere radius=0.01; visual sphere radius=0.01
Joints:
- removed joint fr3_joint8
- added joint touch_tip_joint: type fixed, parent fr3_link7, child touch_tip, origin xyz=0 0 0.15 rpy=0 0 0
